File: Circuitry/Final_PCB/_autosave-Final_PCB.kicad_pcb (KiCad board)
At the start: 2 copper layers, 182.6 x 75.3 mm, 88 parts

Commit message: Photologic board PCB rev1
Changed lines of the file:
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@@
     (tags "mounting hole 3.7mm no annular")
     (attr exclude_from_pos_files exclude_from_bom)
-    (fp_text reference "MOUNT" (at 0 -4.7) (layer "F.SilkS")
+    (fp_text reference "MOUNT" (at 0 -3.7) (layer "F.SilkS")
         (effects (font (size 1 1) (thickness 0.15)))
     )
