File: Circuitry/OG Rig PCB/OG Rig PCB.kicad_sch (KiCad schematic)
At the start: 3 parts, among them U1 SN754410NE, U2 SN754410NE, U3 SN754410NE

Commit message: spout amt test stand
Parts:
- added J1: 5V, symbol Connector:Conn_01x01_Pin
- added J2: GND, symbol Connector:Conn_01x01_Pin
- added J3: Cage, symbol Connector:Conn_01x01_Pin
- added U4, U5: LM311P, P8, symbol LM311P:LM311P
Other:
- moved on the sheet: U1, U2, U3
Changed lines of the file:
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@@
 (kicad_sch (version 20230121) (generator eeschema)
   (paper "A4")
-  (symbol (lib_id "OG PCB LIB:SN754410NE") (at 32.385 27.305 0) (unit 1)
-    (in_bom yes) (on_board yes) (dnp no) (fields_autoplaced)
-    (property "Reference" "U1" (at 90.805 17.78 0)
-      (effects (font (size 1.524 1.524)))
-    )
-    (property "Value" "SN754410NE" (at 90.805 20.32 0)
-      (effects (font (size 1.524 1.524)))
-    )
-    (property "Footprint" "NE16" (at 32.385 27.305 0)
-      (effects (font (size 1.27 1.27) italic) hide)
-    )
-    (property "Datasheet" "SN754410NE" (at 32.385 27.305 0)
+  (symbol (lib_id "Connector:Conn_01x01_Pin") (at 20.955 20.32 0) (unit 1)
+    (in_bom yes) (on_board yes) (dnp no) (fields_autoplaced)
+    (property "Reference" "J1" (at 21.59 15.24 0)
+      (effects (font (size 1.27 1.27)))
+    )
+    (property "Value" "5V" (at 21.59 17.78 0)
+      (effects (font (size 1.27 1.27)))
+    )
+    (property "Footprint" "" (at 20.955 20.32 0)
+      (effects (font (size 1.27 1.27)) hide)
+    )
+    (property "Datasheet" "~" (at 20.955 20.32 0)
+      (effects (font (size 1.27 1.27)) hide)
+    )
+    (pin "1")
+    (instances
+      (project "OG Rig PCB"
+        (path "/8641bd84-d534-4a0d-a208-34ba7fed16d2"
+          (reference "J1") (unit 1)
+        )
+      )
+    )
+  )
+  (symbol (lib_id "Connector:Conn_01x01_Pin") (at 20.955 35.56 0) (unit 1)
+    (in_bom yes) (on_board yes) (dnp no) (fields_autoplaced)
+    (property "Reference" "J3" (at 21.59 31.115 0)
+      (effects (font (size 1.27 1.27)))
+    )
+    (property "Value" "Cage" (at 21.59 33.655 0)
+      (effects (font (size 1.27 1.27)))
+    )
+    (property "Footprint" "" (at 20.955 35.56 0)
+      (effects (font (size 1.27 1.27)) hide)
+    )
+    (property "Datasheet" "~" (at 20.955 35.56 0)
+      (effects (font (size 1.27 1.27)) hide)
+    )
+    (pin "1")
+    (instances
+      (project "OG Rig PCB"
+        (path "/8641bd84-d534-4a0d-a208-34ba7fed16d2"
+          (reference "J3") (unit 1)
+        )
+      )
+    )
+  )
+  (symbol (lib_id "LM311P:LM311P") (at 178.435 42.545 0) (unit 1)
+    (in_bom yes) (on_board yes) (dnp no) (fields_autoplaced)
+    (property "Reference" "U4" (at 216.535 33.02 0)
+      (effects (font (size 1.524 1.524)))
+    )
+    (property "Value" "LM311P" (at 216.535 35.56 0)
+      (effects (font (size 1.524 1.524)))
+    )
+    (property "Footprint" "P8" (at 178.435 42.545 0)
+      (effects (font (size 1.27 1.27) italic) hide)
+    )
+    (property "Datasheet" "LM311P" (at 178.435 42.545 0)
+      (effects (font (size 1.27 1.27) italic) hide)
+    )
+    (pin "1")
+    (pin "2")
+    (pin "3")
+    (pin "4")
+    (pin "5")
+    (pin "6")
+    (pin "7")
+    (pin "8")
+    (instances
+      (project "OG Rig PCB"
+        (path "/8641bd84-d534-4a0d-a208-34ba7fed16d2"
+          (reference "U4") (unit 1)
+        )
+      )
+    )
+  )
+  (symbol (lib_id "Connector:Conn_01x01_Pin") (at 20.955 27.94 0) (unit 1)
+    (in_bom yes) (on_board yes) (dnp no) (fields_autoplaced)
+    (property "Reference" "J2" (at 21.59 22.86 0)
+      (effects (font (size 1.27 1.27)))
+    )
+    (property "Value" "GND" (at 21.59 25.4 0)
+      (effects (font (size 1.27 1.27)))
+    )
+    (property "Footprint" "" (at 20.955 27.94 0)
+      (effects (font (size 1.27 1.27)) hide)
+    )
+    (property "Datasheet" "~" (at 20.955 27.94 0)
+      (effects (font (size 1.27 1.27)) hide)
+    )
+    (pin "1")
+    (instances
+      (project "OG Rig PCB"
+        (path "/8641bd84-d534-4a0d-a208-34ba7fed16d2"
+          (reference "J2") (unit 1)
+        )
+      )
+    )
+  )
+  (symbol (lib_id "OG PCB LIB:SN754410NE") (at 40.64 50.165 0) (unit 1)
+    (in_bom yes) (on_board yes) (dnp no) (fields_autoplaced)
+    (property "Reference" "U1" (at 99.06 40.64 0)
+      (effects (font (size 1.524 1.524)))
+    )
+    (property "Value" "SN754410NE" (at 99.06 43.18 0)
+      (effects (font (size 1.524 1.524)))
+    )
+    (property "Footprint" "NE16" (at 40.64 50.165 0)
+      (effects (font (size 1.27 1.27) italic) hide)
+    )
+    (property "Datasheet" "SN754410NE" (at 40.64 50.165 0)
       (effects (font (size 1.27 1.27) italic) hide)
     )
@@
     )
   )
-  (symbol (lib_id "OG PCB LIB:SN754410NE") (at 31.75 63.5 0) (unit 1)
-    (in_bom yes) (on_board yes) (dnp no) (fields_autoplaced)
-    (property "Reference" "U2" (at 90.17 53.975 0)
-      (effects (font (size 1.524 1.524)))
-    )
-    (property "Value" "SN754410NE" (at 90.17 56.515 0)
-      (effects (font (size 1.524 1.524)))
-    )
-    (property "Footprint" "NE16" (at 31.75 63.5 0)
-      (effects (font (size 1.27 1.27) italic) hide)
-    )
-    (property "Datasheet" "SN754410NE" (at 31.75 63.5 0)
+  (symbol (lib_id "OG PCB LIB:SN754410NE") (at 40.005 86.36 0) (unit 1)
+    (in_bom yes) (on_board yes) (dnp no) (fields_autoplaced)
+    (property "Reference" "U2" (at 98.425 76.835 0)
+      (effects (font (size 1.524 1.524)))
+    )
+    (property "Value" "SN754410NE" (at 98.425 79.375 0)
+      (effects (font (size 1.524 1.524)))
+    )
+    (property "Footprint" "NE16" (at 40.005 86.36 0)
+      (effects (font (size 1.27 1.27) italic) hide)
+    )
+    (property "Datasheet" "SN754410NE" (at 40.005 86.36 0)
       (effects (font (size 1.27 1.27) italic) hide)
     )
@@
     )
   )
-  (symbol (lib_id "OG PCB LIB:SN754410NE") (at 31.75 97.79 0) (unit 1)
-    (in_bom yes) (on_board yes) (dnp no) (fields_autoplaced)
-    (property "Reference" "U3" (at 90.17 88.265 0)
-      (effects (font (size 1.524 1.524)))
-    )
-    (property "Value" "SN754410NE" (at 90.17 90.805 0)
-      (effects (font (size 1.524 1.524)))
-    )
-    (property "Footprint" "NE16" (at 31.75 97.79 0)
-      (effects (font (size 1.27 1.27) italic) hide)
-    )
-    (property "Datasheet" "SN754410NE" (at 31.75 97.79 0)
-      (effects (font (size 1.27 1.27) italic) hide)
-    )
+  (symbol (lib_id "LM311P:LM311P") (at 180.34 91.44 0) (unit 1)
+    (in_bom yes) (on_board yes) (dnp no) (fields_autoplaced)
+    (property "Reference" "U5" (at 218.44 81.28 0)
+      (effects (font (size 1.524 1.524)))
+    )
+    (property "Value" "LM311P" (at 218.44 83.82 0)
+      (effects (font (size 1.524 1.524)))
+    )
+    (property "Footprint" "P8" (at 180.34 91.44 0)
+      (effects (font (size 1.27 1.27) italic) hide)
+    )
+    (property "Datasheet" "LM311P" (at 180.34 91.44 0)
+      (effects (font (size 1.27 1.27) italic) hide)
+    )
+    (pin "1")
+    (pin "2")
+    (pin "3")
+    (pin "4")
+    (pin "5")
+    (pin "6")
+    (pin "7")
+    (pin "8")
+    (instances
+      (project "OG Rig PCB"
+        (path "/8641bd84-d534-4a0d-a208-34ba7fed16d2"
+          (reference "U5") (unit 1)
+        )
+      )
+    )
+  )
+  (symbol (lib_id "OG PCB LIB:SN754410NE") (at 40.005 120.65 0) (unit 1)
+    (in_bom yes) (on_board yes) (dnp no) (fields_autoplaced)
+    (property "Reference" "U3" (at 98.425 111.125 0)
+      (effects (font (size 1.524 1.524)))
+    )
+    (property "Value" "SN754410NE" (at 98.425 113.665 0)
+      (effects (font (size 1.524 1.524)))
+    )
+    (property "Footprint" "NE16" (at 40.005 120.65 0)
+      (effects (font (size 1.27 1.27) italic) hide)
+    )
+    (property "Datasheet" "SN754410NE" (at 40.005 120.65 0)
+      (effects (font (size 1.27 1.27) italic) hide)
+    )
