File: Circuitry/Electrode Tester PCB/Electrode Tester PCB/Electrode Tester PCB.kicad_sch (KiCad schematic)
At the start: 36 parts, among them J19 Conn_01x01_Pin, J20 Conn_01x01_Pin, J21 Conn_01x01_Pin, J22 Conn_01x01_Pin, J23 Conn_01x01_Pin, J24 Conn_01x01_Pin, J25 Conn_01x01_Pin, J26 Conn_01x01_Pin, J27 Conn_01x01_Pin, J28 Conn_01x01_Pin, J29 Conn_01x01_Pin, J30 Conn_01x01_Pin, J31 Conn_01x01_Pin, J32 Conn_01x01_Pin, J33 Conn_01x01_Pin, J34 Conn_01x01_Pin, J35 Conn_01x01_Pin, J36 Conn_01x01_Pin

Commit message: pCb MoUnT
Parts:
- renumbered J21 to CH10_3, CH10_3 to CH10_3_pad1, J22 to CH11_4, CH11_4 to CH11_4_pad1, J23 to CH12_5, CH12_5 to CH12_5_pad1, J24 to CH13_6, CH13_6 to CH13_6_pad1, J25 to CH14_7, CH14_7 to CH14_7_pad1, J26 to CH15_8, CH15_8 to CH15_8_pad1, J27 to CH16_9, CH16_9 to CH16_9_pad1, J29 to CH1_11, CH1_11 to CH1_11_pad1, J30 to CH2_12, CH2_12 to CH2_12_pad1, J31 to CH3_13, CH3_13 to CH3_13_pad1, J32 to CH4_14, CH4_14 to CH4_14_pad1, J33 to CH5_15, CH5_15 to CH5_15_pad1, J34 to CH6_16, CH6_16 to CH6_16_pad1, J35 to CH7_17, CH7_17 to CH7_17_pad1, J36 to CH8_18, CH8_18 to CH8_18_pad1, J20 to CH9_2, CH9_2 to CH9_2_pad1, J28 to GND_10, GND_10 to GND_10_pad1, J19 to R/G_1, R/G1 to R/G_1_pad1
